Commit message: 2025_3_29

File: simulation/urdf/urdf/create_robot.urdf (robot description, URDF)
Before this commit: robot create_robot, 4 links, 3 joints
Links:
- added link back_wheel; visual sphere radius=0.0075
- added link front_wheel; visual sphere radius=0.0075
- link base_link: mass 1 -> None; geometry visual cylinder length=0.08 radius=0.1
- link left_wheel: mass 0.2 -> None; geometry visual cylinder length=0.015 radius=0.0325
- link right_wheel: mass 0.2 -> None; geometry visual cylinder length=0.015 radius=0.0325
Joints:
- added joint back_wheelToBase: type continuous, parent base_link, child back_wheel, origin xyz=-0.08 0 -0.0475 rpy=0 0 0, axis 1 1 1
- added joint front_wheelToBase: type continuous, parent base_link, child front_wheel, origin xyz=0.08 0 -0.0475 rpy=0 0 0, axis 1 1 1
